File: gameboy-breakout-board.kicad_pcb (KiCad board)
At the start: 2 copper layers, 62 x 38 mm, 7 parts, among them J1 GB_GBC_1x32, J2 header

Commit message: Add KiCad logo (copper layer)
Parts:
- added REF**: KiCad-Logo2_6mm_Copper, Symbol:KiCad-Logo2_6mm_Copper, B.Cu at (130.9, 57.4)
