File: gameboy-breakout-board.sch (KiCad schematic (older format))
At the start: 2 parts, among them J1 GB_GBC_1x32, J2 header

Commit message: Update docs
Parts:
- J2: value header -> Header
Changed lines of the file:
@@
 P 3800 2500
 F 0 "J2" H 3850 3417 50  0000 C CNN
-F 1 "header" H 3850 3326 50  0000 C CNN
+F 1 "Header" H 3850 3326 50  0000 C CNN
 F 2 "Connector_PinSocket_2.54mm:PinSocket_2x16_P2.54mm_Vertical" H 3800 2500 50  0001 C CNN
 F 3 "~" H 3800 2500 50  0001 C CNN
